File: PCB/KilnController.kicad_sch (KiCad schematic)
At the start: 32 parts, among them J1 12V 3A PS Header, J10 Display Header, J11 Display Button Header, J12 Moisture Probe 1 Header, J13 Moisture Probe 2 Header, J2 Exhaust Fan Header, J3 Circulation Fan Header, J4 SD Card Module, J5 Exhaust Servo Header, J6 Intake Servo Header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

Commit message: PCB V1 before redesign
Parts:
- added C4, C5: 10uF, Capacitor_THT:CP_Radial_D5.0mm_P2.00mm, symbol Device:C_Polarized_Small_US
- C1, C3: symbol Device:C_Small_US -> Device:C_Small
- D1, D2: value 1N4007 -> 1N5819
Connections:
- net GND: now also C4.2, C5.2
- net PROBE_1_ADC: now also C4.1
- net PROBE_2_ADC: now also C5.1

Commit message: V3 PBC Design
Connections:
- net FAN_CIR_PWM: now also U1.24 (GP18); no longer U1.22 (GP17)
- net FAN_EX_PWM: now also U1.22 (GP17); no longer U1.21 (GP16)
- net HEATER_SSR: now also U1.21 (GP16); no longer U1.24 (GP18)
Changed lines of the file:
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@@
 	)
 	(label "HEATER_SSR"
-		(at 78.74 107.95 0)
+		(at 78.74 115.57 0)
 		(effects
 			(font
@@
 	)
 	(label "FAN_CIR_PWM"
-		(at 78.74 113.03 0)
+		(at 78.74 107.95 0)
 		(effects
 			(font
@@
 	)
 	(label "FAN_EX_PWM"
-		(at 78.74 115.57 0)
-		(effects
-			(font
+		(at 78.74 113.03 0)
+		(effects
+			(font
