File: PCB/KilnController.kicad_pcb (KiCad board)
At the start: 2 copper layers, 133 x 85 mm, 36 parts, among them J1 12V 3A PS Header, J10 Display Header, J11 Display Button Header, J12 Moisture Probe 1 Header, J13 Moisture Probe 2 Header, J2 Exhaust Fan Header, J3 Circulation Fan Header, J4 SD Card Module, J5 Exhaust Servo Header, J6 Intake Servo Header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

Commit message: PCB V1 before redesign
Parts:
- added C4: 10uF, Capacitor_THT:CP_Radial_D5.0mm_P2.00mm, F.Cu at (144.0, 98.0)
- added C5: 10uF, Capacitor_THT:CP_Radial_D5.0mm_P2.00mm, F.Cu at (182.0, 105.0)
- D1, D2: value 1N4007 -> 1N5819
- moved C1 17.1 mm to (147.0, 123.0), turned to -90 degrees
- moved C2 8.06 mm to (140.0, 123.0), turned to 90 degrees
- moved PS1 1.11 mm to (93.4, 123.1)
- moved R2 1.00 mm to (115.0, 84.0)
- moved R3 0.24 mm to (188.6, 73.0)
Routing:
- net /FAN_EX_TACH: track 137.1 -> 92.0 mm, vias 0 -> 1
- net /PROBE_2_ADC: track 96.9 -> 132.3 mm, vias 0 -> 1
- net /FAN_EX_GATE: track 90.9 -> 123.8 mm
- net /+5V_SRC: track 42.8 -> 17.0 mm
- net GND: track 22.9 -> 0.44 mm, vias 0 -> 1
- net /I2C0_SCL: track 163.2 -> 176.3 mm, vias 0 -> 3
- net /LORA_TX: track 77.0 -> 89.1 mm
- net /SD_MISO: track 18.4 -> 10.0 mm
- net /I2C0_SDA: track 173.8 -> 181.6 mm
- net /LORA_CS: track 67.9 -> 75.6 mm, vias 0 -> 1
- net /+12V: track 160.3 -> 153.1 mm
- net /SD_SCK: track 21.6 -> 27.2 mm
- net /SERVO_EXHAUST: track 72.9 -> 78.3 mm, vias 0 -> 2
- net /DISPLAY_RX: track 81.3 -> 76.0 mm
- net /LORA_RST: track 104.9 -> 109.4 mm
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- added copper zone on F.Cu, net GND

Commit message: PCB design V2
Parts:
- moved R2 102.0 mm to (217.0, 83.1), turned to 90 degrees
- moved R7 65.3 mm to (192.9, 120.0)
- moved R6 62.3 mm to (175.9, 120.0)
- moved J11 55.9 mm to (205.5, 146.9)
- moved C4 42.7 mm to (184.0, 113.0), turned to 0 degrees
- moved C3 37.7 mm to (145.0, 90.5)
- moved U4 37.7 mm to (151.8, 95.2)
- moved J10 35.2 mm to (197.1, 147.0), turned to 180 degrees
- moved J9 31.8 mm to (146.5, 64.9)
- moved J6 31.0 mm to (216.0, 129.1), turned to 90 degrees
- moved U3 21.1 mm to (152.8, 131.7)
- moved C1 20.9 mm to (143.0, 143.5)
- moved C5 19.7 mm to (200.0, 113.0)
- moved J13 19.7 mm to (197.9, 102.6)
- moved J12 17.4 mm to (182.5, 102.6)
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Routing:
- net /DISPLAY_BUTTON: track 71.3 -> 177.5 mm, vias 1 -> 3
- net /PROBE_2_DRIVER: track 20.7 -> 87.1 mm
- net /PROBE_1_DRIVER: track 9.27 -> 72.7 mm
- net /LORA_RST: track 109.4 -> 51.8 mm
- net /+5V: track 295.1 -> 347.2 mm, vias 0 -> 2
- net /LORA_SCK: track 88.4 -> 38.3 mm, vias 1 -> 0
- net /LORA_TX: track 89.1 -> 49.9 mm, vias 0 -> 1
- net /SERVO_EXHAUST: track 78.3 -> 114.3 mm
- net /FAN_EX_TACH: track 92.0 -> 127.1 mm, vias 1 -> 2
- net /LORA_RX: track 66.7 -> 32.1 mm
- net /LORA_CS: track 75.6 -> 44.0 mm, vias 1 -> 0
- net /+3V3: track 107.0 -> 131.3 mm
- net /PROBE_1_ADC: track 77.6 -> 97.6 mm
- net /FAN_CIR_GATE: track 38.6 -> 56.8 mm, vias 0 -> 2
- net /SD_SCK: track 27.2 -> 9.20 mm
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Other:
- board size 133 x 85 mm -> 143 x 95 mm

Commit message: V3 PBC Design
Parts:
- moved J11 82.0 mm to (203.5, 64.9)
- moved J9 35.7 mm to (144.1, 100.5), turned to -90 degrees
- moved J6 20.1 mm to (197.1, 136.0), turned to 180 degrees
- moved D1 18.7 mm to (171.3, 72.8)
- moved D2 18.7 mm to (141.3, 72.8)
- moved J2 18.7 mm to (177.1, 64.9)
- moved J3 18.7 mm to (144.7, 64.8)
- moved Q1 18.7 mm to (180.3, 79.8)
- moved Q2 18.7 mm to (150.3, 79.9)
- moved R1 18.7 mm to (192.0, 72.8)
- moved R2 18.7 mm to (198.3, 83.0)
- moved R3 18.7 mm to (186.3, 72.9)
- moved R4 18.7 mm to (157.1, 83.1)
- moved R5 18.7 mm to (163.1, 83.1)
- moved J5 17.5 mm to (206.9, 89.6)
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Connections:
- U1 pad 21: /FAN_EX_PWM -> /HEATER_SSR
- U1 pad 22: /FAN_CIR_PWM -> /FAN_EX_PWM
- U1 pad 24: /HEATER_SSR -> /FAN_CIR_PWM
Routing:
- net /DISPLAY_BUTTON: track 177.5 -> 105.0 mm, vias 3 -> 1
- net /SERVO_INTAKE: track 94.9 -> 62.4 mm
- net /HEATER_SSR: track 38.6 -> 12.2 mm
- net /FAN_EX_GATE: track 113.2 -> 90.5 mm, vias 2 -> 0
- net /FAN_EX_TACH: track 127.1 -> 106.9 mm, vias 2 -> 0
- net /+12V: track 171.0 -> 152.3 mm
- net /PROBE_1_ADC: track 97.6 -> 115.2 mm
- net /FAN_EX_PWM: track 105.6 -> 88.9 mm
- net /FAN_CIR_GATE: track 56.8 -> 40.4 mm, vias 2 -> 1
- net /PROBE_2_ADC: track 117.1 -> 128.1 mm
- net /FAN_CIR_PWM: track 59.7 -> 70.4 mm, vias 0 -> 2
- net /+5V: track 347.2 -> 356.2 mm
- net /LORA_RST: track 51.8 -> 59.4 mm
- net /+3V3: track 131.3 -> 123.7 mm
- net /PROBE_1_DRIVER: track 72.7 -> 78.9 mm, vias 0 -> 2
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Other:
- board size 143 x 95 mm -> 140 x 95 mm

Commit message: Final PCB for manufacturing
Other:
- board text added: "(c) Steve Elias 2026"
- board text added: "KS Kiln v1.0"
